File: hw/3dglassbox.kicad_sch (KiCad schematic)
At the start: 72 parts, among them J1 SGI stereo, J2 SGI Impact stereo, J3 12v DC, J4 AVR-ISP-6, J6 VESA, J7 VSYNC, J8 ASUS VR-100, Q1 2N7002, Q2 2N7002, SW1 vsync_flip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

Commit message: pcb design done
Parts:
- removed C7: 0.1uF, Capacitor_SMD:C_0805_2012Metric_Pad1.18x1.45mm_HandSolder, symbol Device:C
- added D18: LED, LED_THT:LED_D5.0mm, symbol Device:LED
- added H1, H2, H3, H4: MountingHole_Pad, MountingHole:MountingHole_3.2mm_M3_Pad, symbol Mechanical:MountingHole_Pad
- added R21: 1K, Resistor_SMD:R_0805_2012Metric_Pad1.20x1.40mm_HandSolder, symbol Device:R
- added SW5: SW_SEL, Button_Switch_SMD:SW_Push_1P1T_NO_6x6mm_H9.5mm, symbol Switch:SW_Push
- added SW6: SW_NEXT, Button_Switch_SMD:SW_Push_1P1T_NO_6x6mm_H9.5mm, symbol Switch:SW_Push
- R17, R18, R19, R20: value 4k7 -> 4K7
Connections:
- net B1: now also R21.1
- net B2: now also SW5.1
- net B3: now also SW6.1
- net GND: now also D18.1 (K), H1.1, H2.1, H3.1, H4.1, SW5.2, SW6.2
- new net: D18.2 (A), R21.2
Other:
- note added: "SW5/SW6: select IR emitter mode"
- moved on the sheet: C3, C4, C5, C6, J4, Q2, R17, SW2, TP1, TP2, TP3, TP4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
